Commit message: Setup simulation

File: description/robot_core.xacro (robot description, xacro)
@@ -41,4 +41,7 @@
         </xacro:inertial_cylinder>
     </link>
+    <gazebo reference="chassis">
+        <material>Gazebo/White</material>
+    </gazebo>
     <!-- Left Wheel Link-->
     <joint name="left_wheel_joint" type="continuous">
@@ -66,4 +69,7 @@
         </xacro:inertial_cylinder>
     </link>
+    <gazebo reference="left_wheel">
+        <material>Gazebo/Blue</material>
+    </gazebo>
     <!-- right Wheel Link-->
     <joint name="right_wheel_joint" type="continuous">
@@ -91,4 +97,7 @@
         </xacro:inertial_cylinder>
     </link>
+    <gazebo reference="right_wheel">
+        <material>Gazebo/Blue</material>
+    </gazebo>
     <!-- caster Wheel link -->
     <joint name="caster_wheel_joint_back" type="fixed">
@@ -115,4 +124,9 @@
         </xacro:inertial_sphere>
     </link>
+    <gazebo reference="caster_wheel_back">
+        <material>Gazebo/Black</material>
+        <mu1 value="0.001"/>
+        <mu2 value="0.001"/>
+    </gazebo>
     <!-- caster Wheel link -->
     <joint name="caster_wheel_joint" type="fixed">
@@ -139,3 +153,8 @@
         </xacro:inertial_sphere>
     </link>
+    <gazebo reference="caster_wheel">
+        <material>Gazebo/Black</material>
+        <mu1 value="0.001"/>
+        <mu2 value="0.001"/>
+    </gazebo>
 </robot>
