Commit message: test

File: description/robot.urdf.xacro (robot description, xacro)
@@ -1,5 +1,11 @@
 <?xml version="1.0"?>
 <robot xmlns:xacro="http://www.ros.org/wiki/xacro"  name="robot">
+    <xacro:arg name="use_ros2_control" default="true"/>
     <xacro:include filename="robot_core.xacro"/>
-    <xacro:include filename="gazebo_control.xacro"/>
+    <xacro:if value="$(arg use_ros2_control)">
+        <xacro:include filename="ros2_control.xacro"/>
+    </xacro:if>
+    <xacro:unless value="$(arg use_ros2_control)">
+        <xacro:include filename="gazebo_control.xacro"/>
+    </xacro:unless>
 </robot>

File: description/robot_core.xacro (robot description, xacro)
@@ -62,5 +62,5 @@
             <origin xyz="0 0 0"/>
             <geometry>
-                <cylinder radius="0.031" length="0.006"/>
+                <sphere radius="0.031" />
             </geometry>
         </collision>
@@ -90,5 +90,5 @@
             <origin xyz="0 0 0"/>
             <geometry>
-                <cylinder radius="0.031" length="0.006"/>
+                <sphere radius="0.031"/>
             </geometry>
         </collision>
